Commit message: adapted name

File: beckhoff_ads_bringup/urdf/beckhoff_bot/beckhoff_ads_interfaces.ros2_control.xacro (robot description, xacro)
@@ -1,5 +1,5 @@
 <?xml version="1.0" encoding="UTF-8"?>
 <robot xmlns:xacro="http://wiki.ros.org/xacro">
-    <xacro:macro name="command_interface_PLC" params="name initial_value:='' PLC_symbol PLC_type n_elements:=1 index:=''">
+    <xacro:macro name="command_to_PLC" params="name initial_value:='' PLC_symbol PLC_type n_elements:=1 index:=''">
         <command_interface name="${name}">
             <xacro:if value="${initial_value != ''}">
@@ -14,5 +14,5 @@
         </command_interface>
     </xacro:macro>
-    <xacro:macro name="state_interface_PLC" params="name PLC_symbol PLC_type n_elements:=1 index:=''">
+    <xacro:macro name="state_from_PLC" params="name PLC_symbol PLC_type n_elements:=1 index:=''">
         <state_interface name="${name}">
             <param name="PLC_symbol">${PLC_symbol}</param>
